Commit message: fix the bug of root_pos and complete the xarm7 set

File: thirdparty/ManiSkill/mani_skill/assets/robots/xarm6/xarm6_allegro_right.urdf (robot description, URDF)
Before this commit: robot xarm6_allegro, 31 links, 30 joints
Links:
- link base_link: geometry collision box size=0.0414 0.0538 0.0428; collision box size=0.0414 0.0720 0.013
- link link_0: geometry collision box size=0.0196 0.0275 0.0164; visual mesh filename=../allegro_hand/meshes/visual/link_0.0.glb
- link link_1: geometry collision box size=0.0196 0.0275 0.054; visual mesh filename=../allegro_hand/meshes/visual/link_1.0.glb
- link link_10: geometry collision box size=0.0196 0.0275 0.0384; visual mesh filename=../allegro_hand/meshes/visual/link_2.0.glb
- link link_11: geometry collision box size=0.0196 0.0269 0.022; visual mesh filename=../allegro_hand/meshes/visual/link_3.0.glb
- link link_11_tip: geometry collision mesh filename=../allegro_hand/meshes/collision/link_tip.obj; visual mesh filename=../allegro_hand/meshes/visual/link_tip.glb
- link link_12: geometry collision box size=0.0358 0.034 0.0455; visual mesh filename=../allegro_hand/meshes/visual/link_12.0_right.glb
- link link_13: geometry collision box size=0.0196 0.0275 0.0177; visual mesh filename=../allegro_hand/meshes/visual/link_13.0.glb
- link link_14: geometry collision box size=0.0196 0.0275 0.0514; visual mesh filename=../allegro_hand/meshes/visual/link_14.0.glb
- link link_15: geometry collision box size=0.0196 0.0269 0.04; visual mesh filename=../allegro_hand/meshes/visual/link_15.0.glb
- link link_15_tip: geometry collision mesh filename=../allegro_hand/meshes/collision/link_tip.obj; visual mesh filename=../allegro_hand/meshes/visual/link_tip.glb
- link link_2: geometry collision box size=0.0196 0.0275 0.0384; visual mesh filename=../allegro_hand/meshes/visual/link_2.0.glb
- link link_3: geometry collision box size=0.0196 0.0269 0.022; visual mesh filename=../allegro_hand/meshes/visual/link_3.0.glb
- link link_3_tip: geometry collision mesh filename=../allegro_hand/meshes/collision/link_tip.obj; visual mesh filename=../allegro_hand/meshes/visual/link_tip.glb
- link link_4: geometry collision box size=0.0196 0.0275 0.0164; visual mesh filename=../allegro_hand/meshes/visual/link_0.0.glb
- link link_5: geometry collision box size=0.0196 0.0275 0.054; visual mesh filename=../allegro_hand/meshes/visual/link_1.0.glb
- link link_6: geometry collision box size=0.0196 0.0275 0.0384; visual mesh filename=../allegro_hand/meshes/visual/link_2.0.glb
- link link_7: geometry collision box size=0.0196 0.0269 0.022; visual mesh filename=../allegro_hand/meshes/visual/link_3.0.glb
- link link_7_tip: geometry collision mesh filename=../allegro_hand/meshes/collision/link_tip.obj; visual mesh filename=../allegro_hand/meshes/visual/link_tip.glb
- link link_8: geometry collision box size=0.0196 0.0275 0.0164; visual mesh filename=../allegro_hand/meshes/visual/link_0.0.glb
- link link_9: geometry collision box size=0.0196 0.0275 0.054; visual mesh filename=../allegro_hand/meshes/visual/link_1.0.glb

File: thirdparty/ManiSkill/mani_skill/assets/robots/xarm7/xarm7_shadow_right.urdf (robot description, URDF)
Before this commit: robot xarm7, 40 links, 39 joints
Joints:
- joint joint_eef: origin xyz=0 0 0 rpy=0 0 3.1416 -> xyz=0 0 0 rpy=0 0 1.57079
