Commit message: complete the ur5e set and add the iiwa+allegro

File: thirdparty/ManiSkill/mani_skill/assets/robots/iiwa7/iiwa7_allegro_right.urdf (robot description, URDF)
Before this commit: robot xarm7, 31 links, 30 joints
Links:
- removed link link1
- removed link link2
- removed link link3
- removed link link4
- removed link link5
- removed link link6
- removed link link7
- removed link link_base
- added link link_0_arm, mass 4.855658; collision mesh filename=meshes/collision/link_0.obj; visual mesh filename=meshes/visual/link_0.glb
- added link link_1_arm, mass 3.394011; collision mesh filename=meshes/collision/link_1.obj; visual mesh filename=meshes/visual/link_1.glb
- added link link_2_arm, mass 4.031991; collision mesh filename=meshes/collision/link_2.obj; visual mesh filename=meshes/visual/link_2.glb
- added link link_3_arm, mass 3.394011; collision mesh filename=meshes/collision/link_3.obj; visual mesh filename=meshes/visual/link_3.glb
- added link link_4_arm, mass 4.031989; collision mesh filename=meshes/collision/link_4.obj; visual mesh filename=meshes/visual/link_4.glb
- added link link_5_arm, mass 1.529239; collision mesh filename=meshes/collision/link_5.obj; visual mesh filename=meshes/visual/link_5.glb
- added link link_6_arm, mass 2.403626; collision mesh filename=meshes/collision/link_6.obj; visual mesh filename=meshes/visual/link_6.glb
- added link link_7_arm, mass 0.259474; collision mesh filename=meshes/collision/link_7.obj; visual mesh filename=meshes/visual/link_7.glb
Joints:
- removed joint joint1
- removed joint joint2
- removed joint joint3
- removed joint joint4
- removed joint joint5
- removed joint joint6
- removed joint joint7
- added joint A1: type revolute, parent link_0_arm, child link_1_arm, origin xyz=0.0 0.0 0.1475 rpy=0 0 0, axis 0.0 0.0 1.0, limit lower=-2.96705972839 upper=2.96705972839 effort=200 velocity=1.71042266695
- added joint A2: type revolute, parent link_1_arm, child link_2_arm, origin xyz=0.0 -0.0105 0.1925 rpy=0 0 0, axis 0.0 1.0 0.0, limit lower=-2.09439510239 upper=2.09439510239 effort=200 velocity=1.71042266695
- added joint A3: type revolute, parent link_2_arm, child link_3_arm, origin xyz=0.0 0.0105 0.2075 rpy=0 0 0, axis 0.0 0.0 1.0, limit lower=-2.96705972839 upper=2.96705972839 effort=200 velocity=1.74532925199
- added joint A4: type revolute, parent link_3_arm, child link_4_arm, origin xyz=0.0 0.0105 0.1925 rpy=0 0 0, axis 0.0 -1.0 0.0, limit lower=-2.09439510239 upper=2.09439510239 effort=200 velocity=2.26892802759
- added joint A5: type revolute, parent link_4_arm, child link_5_arm, origin xyz=0.0 -0.0105 0.2075 rpy=0 0 0, axis 0.0 0.0 1.0, limit lower=-2.96705972839 upper=2.96705972839 effort=200 velocity=2.44346095279
- added joint A6: type revolute, parent link_5_arm, child link_6_arm, origin xyz=0.0 -0.0707 0.1925 rpy=0 0 0, axis 0.0 1.0 0.0, limit lower=-2.09439510239 upper=2.09439510239 effort=200 velocity=3.14159265359
- added joint A7: type revolute, parent link_6_arm, child link_7_arm, origin xyz=0.0 0.0707 0.091 rpy=0 0 0, axis 0.0 0.0 1.0, limit lower=-3.05432619099 upper=3.05432619099 effort=200 velocity=3.14159265359
- joint joint_eef: origin xyz=0 0 0.095 rpy=0 0 3.1416 -> xyz=0 0 0.13 rpy=0 0 0; parent link7 -> link_7_arm

File: thirdparty/ManiSkill/mani_skill/assets/robots/ur5e/ur5e_allegro_right.urdf (robot description, URDF)
Before this commit: robot xarm7, 31 links, 30 joints
Links:
- removed link link1
- removed link link2
- removed link link3
- removed link link4
- removed link link5
- removed link link6
- removed link link7
- removed link link_base
- added link base
- added link base_link
- added link base_link_inertia, mass 4.0; collision mesh filename=meshes/collision/base.obj; visual mesh filename=meshes/visual/base.glb
- added link ee_link
- added link forearm_link, mass 2.275; collision mesh filename=meshes/collision/forearm.obj; visual mesh filename=meshes/visual/forearm.glb
- added link shoulder_link, mass 3.7; collision mesh filename=meshes/collision/shoulder.obj; visual mesh filename=meshes/visual/shoulder.glb
- added link upper_arm_link, mass 8.393; collision mesh filename=meshes/collision/upperarm.obj; visual mesh filename=meshes/visual/upperarm.glb
- added link wrist_1_link, mass 1.219; collision mesh filename=meshes/collision/wrist1.obj; visual mesh filename=meshes/visual/wrist1.glb
- added link wrist_2_link, mass 1.219; collision mesh filename=meshes/collision/wrist2.obj; visual mesh filename=meshes/visual/wrist2.glb
- added link wrist_3_link, mass 0.1879; collision mesh filename=meshes/collision/wrist3.obj; visual mesh filename=meshes/visual/wrist3.glb
Joints:
- removed joint joint1
- removed joint joint2
- removed joint joint3
- removed joint joint4
- removed joint joint5
- removed joint joint6
- removed joint joint7
- removed joint joint_eef
- added joint base_link-base_fixed_joint: type fixed, parent base_link, child base, origin xyz=0 0 0 rpy=0 0 3.14159265359
- added joint base_link-base_link_inertia: type fixed, parent base_link, child base_link_inertia, origin xyz=0 0 0 rpy=0 0 3.14159265359
- added joint elbow_joint: type revolute, parent upper_arm_link, child forearm_link, origin xyz=-0.425 0 0 rpy=0 0 0, axis 0 0 1, limit lower=-3.14159265359 upper=3.14159265359 effort=150.0 velocity=3.14159265359
- added joint mount_joint: type fixed, parent wrist_3_link, child base_link_hand, origin xyz=0.0 0.0 0.095 rpy=0 0 -1.57079
- added joint shoulder_lift_joint: type revolute, parent shoulder_link, child upper_arm_link, origin xyz=0 0 0 rpy=1.570796327 0 0, axis 0 0 1, limit lower=-6.28318530718 upper=6.28318530718 effort=150.0 velocity=3.14159265359
- added joint shoulder_pan_joint: type revolute, parent base_link_inertia, child shoulder_link, origin xyz=0 0 0.1625 rpy=0 0 0, axis 0 0 1, limit lower=-6.28318530718 upper=6.28318530718 effort=150.0 velocity=3.14159265359
- added joint wrist_1_joint: type revolute, parent forearm_link, child wrist_1_link, origin xyz=-0.3922 0 0.1333 rpy=0 0 0, axis 0 0 1, limit lower=-6.28318530718 upper=6.28318530718 effort=28.0 velocity=3.14159265359
- added joint wrist_2_joint: type revolute, parent wrist_1_link, child wrist_2_link, origin xyz=0 -0.0997 -2.0448811823e-11 rpy=1.570796327 0 0, axis 0 0 1, limit lower=-6.28318530718 upper=6.28318530718 effort=28.0 velocity=3.14159265359
- added joint wrist_3-flange: type fixed, parent wrist_3_link, child ee_link, origin xyz=0 0 0 rpy=0 0 -1.5707926
- added joint wrist_3_joint: type revolute, parent wrist_2_link, child wrist_3_link, origin xyz=0 0.0996 -2.04283014801e-11 rpy=1.57079632659 3.14159265359 3.14159265359, axis 0 0 1, limit lower=-6.28318530718 upper=6.28318530718 effort=28.0 velocity=3.14159265359

File: thirdparty/ManiSkill/mani_skill/assets/robots/ur5e/ur5e_leap_right.urdf (robot description, URDF)
Before this commit: robot xarm7, 30 links, 29 joints
Links:
- removed link link1
- removed link link2
- removed link link3
- removed link link4
- removed link link5
- removed link link6
- removed link link7
- removed link link_base
- added link base
- added link base_link
- added link base_link_inertia, mass 4.0; collision mesh filename=meshes/collision/base.obj; visual mesh filename=meshes/visual/base.glb
- added link ee_link
- added link forearm_link, mass 2.275; collision mesh filename=meshes/collision/forearm.obj; visual mesh filename=meshes/visual/forearm.glb
- added link shoulder_link, mass 3.7; collision mesh filename=meshes/collision/shoulder.obj; visual mesh filename=meshes/visual/shoulder.glb
- added link upper_arm_link, mass 8.393; collision mesh filename=meshes/collision/upperarm.obj; visual mesh filename=meshes/visual/upperarm.glb
- added link wrist_1_link, mass 1.219; collision mesh filename=meshes/collision/wrist1.obj; visual mesh filename=meshes/visual/wrist1.glb
- added link wrist_2_link, mass 1.219; collision mesh filename=meshes/collision/wrist2.obj; visual mesh filename=meshes/visual/wrist2.glb
- added link wrist_3_link, mass 0.1879; collision mesh filename=meshes/collision/wrist3.obj; visual mesh filename=meshes/visual/wrist3.glb
Joints:
- removed joint joint1
- removed joint joint2
- removed joint joint3
- removed joint joint4
- removed joint joint5
- removed joint joint6
- removed joint joint7
- removed joint joint_eef
- added joint base_link-base_fixed_joint: type fixed, parent base_link, child base, origin xyz=0 0 0 rpy=0 0 3.14159265359
- added joint base_link-base_link_inertia: type fixed, parent base_link, child base_link_inertia, origin xyz=0 0 0 rpy=0 0 3.14159265359
- added joint elbow_joint: type revolute, parent upper_arm_link, child forearm_link, origin xyz=-0.425 0 0 rpy=0 0 0, axis 0 0 1, limit lower=-3.14159265359 upper=3.14159265359 effort=150.0 velocity=3.14159265359
- added joint mount_joint: type fixed, parent wrist_3_link, child base_hand, origin xyz=0.0 0.0 0.0 rpy=0 0 -1.57079
- added joint shoulder_lift_joint: type revolute, parent shoulder_link, child upper_arm_link, origin xyz=0 0 0 rpy=1.570796327 0 0, axis 0 0 1, limit lower=-6.28318530718 upper=6.28318530718 effort=150.0 velocity=3.14159265359
- added joint shoulder_pan_joint: type revolute, parent base_link_inertia, child shoulder_link, origin xyz=0 0 0.1625 rpy=0 0 0, axis 0 0 1, limit lower=-6.28318530718 upper=6.28318530718 effort=150.0 velocity=3.14159265359
- added joint wrist_1_joint: type revolute, parent forearm_link, child wrist_1_link, origin xyz=-0.3922 0 0.1333 rpy=0 0 0, axis 0 0 1, limit lower=-6.28318530718 upper=6.28318530718 effort=28.0 velocity=3.14159265359
- added joint wrist_2_joint: type revolute, parent wrist_1_link, child wrist_2_link, origin xyz=0 -0.0997 -2.0448811823e-11 rpy=1.570796327 0 0, axis 0 0 1, limit lower=-6.28318530718 upper=6.28318530718 effort=28.0 velocity=3.14159265359
- added joint wrist_3-flange: type fixed, parent wrist_3_link, child ee_link, origin xyz=0 0 0 rpy=0 0 -1.5707926
- added joint wrist_3_joint: type revolute, parent wrist_2_link, child wrist_3_link, origin xyz=0 0.0996 -2.04283014801e-11 rpy=1.57079632659 3.14159265359 3.14159265359, axis 0 0 1, limit lower=-6.28318530718 upper=6.28318530718 effort=28.0 velocity=3.14159265359

File: thirdparty/ManiSkill/mani_skill/assets/robots/xarm6/xarm6_allegro_left.urdf (robot description, URDF)
Before this commit: robot xarm6, 31 links, 30 joints
Links:
- removed link base_link
- added link base_link_hand, mass 0.4154; collision box size=0.0414 0.0538 0.0428; collision box size=0.0414 0.0720 0.013
Joints:
- joint gripper_base_joint: child base_link -> base_link_hand
- joint joint_0.0: parent base_link -> base_link_hand
- joint joint_12.0: parent base_link -> base_link_hand
- joint joint_4.0: parent base_link -> base_link_hand
- joint joint_8.0: parent base_link -> base_link_hand
- joint palm_joint: parent base_link -> base_link_hand

File: thirdparty/ManiSkill/mani_skill/assets/robots/xarm6/xarm6_allegro_right.urdf (robot description, URDF)
Before this commit: robot xarm6_allegro, 31 links, 30 joints
Links:
- removed link base_link
- added link base_link_hand, mass 0.4154; collision box size=0.0414 0.0538 0.0428; collision box size=0.0414 0.0720 0.013
Joints:
- joint gripper_base_joint: child base_link -> base_link_hand
- joint joint_0: parent base_link -> base_link_hand
- joint joint_12: parent base_link -> base_link_hand
- joint joint_4: parent base_link -> base_link_hand
- joint joint_8: parent base_link -> base_link_hand
- joint palm_joint: parent base_link -> base_link_hand
