Commit message: optimize the init pos and add ur5e+allegro and the camera binding to four types of hand

File: thirdparty/ManiSkill/mani_skill/assets/robots/franka/panda.urdf (robot description, URDF)
Before this commit: robot panda, 16 links, 15 joints
Links:
- removed link panda_left_hand
Joints:
- removed joint panda_left_hand_joint

Commit message: tune param to complete the peg insertion task

File: thirdparty/ManiSkill/mani_skill/assets/robots/franka/panda.urdf (robot description, URDF)
Before this commit: robot panda, 15 links, 14 joints
Links:
- added link camera_base_link
- added link camera_link, mass 0.564; collision box size=0.02005 0.099 0.023; visual mesh filename=realsense2_description/meshes/d415.stl
Joints:
- added joint camera_link_joint: type fixed, parent camera_base_link, child camera_link, origin xyz=0 0.02 0.0115 rpy=0 0 0
- added joint realsense_joint: type fixed, parent panda_hand, child camera_base_link, origin xyz=-0.035 0 0.036 rpy=0 -1.5707 0

File: thirdparty/ManiSkill/mani_skill/assets/robots/xarm7/xarm7_allegro_right.urdf (robot description, URDF)
Before this commit: robot xarm7, 31 links, 30 joints
Joints:
- joint joint_eef: origin xyz=0 0 0.095 rpy=0 0 3.1416 -> xyz=0 0 0.095 rpy=0 0 0
