Commit message: add virtual link of leap for retargeting and use different seed when collect with teleoperate

File: thirdparty/ManiSkill/mani_skill/assets/robots/xarm7/xarm7_leap_right.urdf (robot description, URDF)
Before this commit: robot xarm7, 30 links, 29 joints
Links:
- added link palm
Joints:
- added joint palm_joint: type fixed, parent base_hand, child palm, origin xyz=0 0 -0.088 rpy=0 0 0
