Commit message: urdf, task solution, init state of robbot in faucet_env

File: thirdparty/ManiSkill/mani_skill/assets/my_faucet/faucet_pack/mobility.urdf (robot description, URDF)
Before this commit: robot partnet_1c684a5a113c4536b7a867e9b35a1295, 3 links, 2 joints
Links:
- removed link base
- removed link link_0
- removed link link_1
- added link base_link, mass 0.1; collision cylinder length=0.005 radius=0.05; visual cylinder length=0.005 radius=0.05
- added link global_base
- added link handle_link, mass 0.001; collision cylinder length=0.12 radius=0.0045; visual cylinder length=0.12 radius=0.0045
- added link main_body, mass 0.2; collision cylinder length=0.13 radius=0.025; visual cylinder length=0.13 radius=0.025
- added link spout_link, mass 0.1; collision cylinder length=0.02 radius=0.015; collision cylinder length=0.13 radius=0.02
- added link top_link, mass 0.1; collision cylinder length=0.04 radius=0.025; visual cylinder length=0.04 radius=0.025
Joints:
- removed joint joint_0
- removed joint joint_1
- added joint global_rotation: type fixed, parent global_base, child base_link, origin xyz=0 0 0 rpy=0 0 3.14159
- added joint joint_base_to_body: type fixed, parent base_link, child main_body, origin xyz=0 0 0.005 rpy=0 0 0
- added joint joint_body_to_spout: type fixed, parent main_body, child spout_link, origin xyz=0 0 0.08 rpy=0 0 0
- added joint joint_body_to_top: type revolute, parent main_body, child top_link, origin xyz=0 0 0.13 rpy=0 0 0, axis 0 0 1, limit lower=-1.7 upper=1.7 effort=5.0 velocity=2.0
- added joint joint_top_to_handle: type fixed, parent top_link, child handle_link, origin xyz=0 0 0.025 rpy=0 0 0

File: thirdparty/ManiSkill/mani_skill/assets/my_laptop/laptop_pack2/mobility.urdf (robot description, URDF)
Before this commit: robot partnet_cc0535a34cdc7d676bf98d15712168f, 3 links, 2 joints
Links:
- removed link base
- removed link link_0
- removed link link_1
- added link base_link, mass 1.0; collision box size=0.30 0.20 0.02; visual box size=0.30 0.20 0.02
- added link global_base
- added link screen_link, mass 0.1; collision box size=0.30 0.005 0.20; visual box size=0.30 0.005 0.20
Joints:
- removed joint joint_0
- removed joint joint_1
- added joint global_rotation: type fixed, parent global_base, child base_link, origin xyz=0 0 0 rpy=0 0 1.5708
- added joint hinge_joint: type revolute, parent base_link, child screen_link, origin xyz=0 -0.10 0.02 rpy=0 0 0, axis 1 0 0, limit lower=-1.57 upper=1.57 effort=4.0 velocity=2.0
