Commit message: remodify urdf and leap friction

File: thirdparty/ManiSkill/mani_skill/assets/my_laptop/laptop_pack2/mobility.urdf (robot description, URDF)
Before this commit: robot laptop_model_single_hinge_corrected, 3 links, 2 joints
Links:
- link screen_link: mass 0.1 -> 0.05; geometry collision box size=0.30 0.01 0.20; visual box size=0.30 0.01 0.20
