Commit message: add allegro aux link

File: thirdparty/ManiSkill/mani_skill/assets/robots/ur5e/ur5e_allegro_right.urdf (robot description, URDF)
Before this commit: robot ur5e_shadow_right, 33 links, 32 joints
Links:
- added link base_link_hand_aux0
- added link base_link_hand_aux1
- added link base_link_hand_aux2
- added link link_11_tip_aux0
- added link link_11_tip_aux1
- added link link_11_tip_aux2
- added link link_15_tip_aux0
- added link link_15_tip_aux1
- added link link_15_tip_aux2
- added link link_3_tip_aux0
- added link link_3_tip_aux1
- added link link_3_tip_aux2
- added link link_7_tip_aux0
- added link link_7_tip_aux1
- added link link_7_tip_aux2
Joints:
- added joint base_link_hand_aux0_joint: type fixed, parent base_link_hand, child base_link_hand_aux0, origin xyz=0.2 0 0 rpy=0 0 0
- added joint base_link_hand_aux1_joint: type fixed, parent base_link_hand, child base_link_hand_aux1, origin xyz=0.0 0.2 0 rpy=0 0 0
- added joint base_link_hand_aux2_joint: type fixed, parent base_link_hand, child base_link_hand_aux2, origin xyz=0.0 0.0 0.2 rpy=0 0 0
- added joint link_11_tip_aux0_joint: type fixed, parent link_11_tip, child link_11_tip_aux0, origin xyz=0.2 0 0 rpy=0 0 0
- added joint link_11_tip_aux1_joint: type fixed, parent link_11_tip, child link_11_tip_aux1, origin xyz=0.0 0.2 0 rpy=0 0 0
- added joint link_11_tip_aux2_joint: type fixed, parent link_11_tip, child link_11_tip_aux2, origin xyz=0.0 0.0 0.2 rpy=0 0 0
- added joint link_15_tip_aux0_joint: type fixed, parent link_15_tip, child link_15_tip_aux0, origin xyz=0.2 0 0 rpy=0 0 0
- added joint link_15_tip_aux1_joint: type fixed, parent link_15_tip, child link_15_tip_aux1, origin xyz=0.0 0.2 0 rpy=0 0 0
- added joint link_15_tip_aux2_joint: type fixed, parent link_15_tip, child link_15_tip_aux2, origin xyz=0.0 0.0 0.2 rpy=0 0 0
- added joint link_3_tip_aux0_joint: type fixed, parent link_3_tip, child link_3_tip_aux0, origin xyz=0.2 0 0 rpy=0 0 0
- added joint link_3_tip_aux1_joint: type fixed, parent link_3_tip, child link_3_tip_aux1, origin xyz=0.0 0.2 0 rpy=0 0 0
- added joint link_3_tip_aux2_joint: type fixed, parent link_3_tip, child link_3_tip_aux2, origin xyz=0.0 0.0 0.2 rpy=0 0 0
- added joint link_7_tip_aux0_joint: type fixed, parent link_7_tip, child link_7_tip_aux0, origin xyz=0.2 0 0 rpy=0 0 0
- added joint link_7_tip_aux1_joint: type fixed, parent link_7_tip, child link_7_tip_aux1, origin xyz=0.0 0.2 0 rpy=0 0 0
- added joint link_7_tip_aux2_joint: type fixed, parent link_7_tip, child link_7_tip_aux2, origin xyz=0.0 0.0 0.2 rpy=0 0 0
